File: stem.brd (EAGLE design)
At the start: 76.2 x 69.9 mm, 3 parts, among them J1 BG300-02-X-X-A_REVC

Commit message: fridge_magnet pcb files
Routing:
- net GND: track 13.8 -> 0.00 mm
Other:
- board size 76.2 x 69.9 mm -> 76.2 x 77.8 mm
