File: magnet.brd (EAGLE design)
At the start: 76.2 x 76.2 mm, 37 parts, among them U1 IN100, U2 LTC3106EFE#PBF, U3 BME280, U4 SGP30, Y1 CX3225SB26000D0FLJCC, Y2 ECS-.327-12.5-16-TR

Commit message: File check-in
Parts:
- added C19: 100nF, OPL_Capacitor:C0603
- added H1: MOUNT-HOLE3.0, holes:3,0
- added R4, R5: 2.2K, SparkFun-Resistors:0603
- moved C18 124.3 mm to (24.5, 5.59), turned to 270 degrees
- moved C17 119.0 mm to (24.5, 3.73), turned to 270 degrees
- moved U4 109.7 mm to (20.5, 0.48), turned to 180 degrees
- moved U3 108.3 mm to (20.7, 4.98), turned to 180 degrees
- moved C10 20.4 mm to (2.79, 10.0)
- moved C11 20.4 mm to (0.89, 10.0)
- moved C9 20.4 mm to (4.70, 10.0)
- moved L2 14.2 mm to (-8.81, 10.4)
- moved U2 14.2 mm to (-8.76, 4.45)
- moved R2 14.0 mm to (-2.54, 4.06)
- moved R3 14.0 mm to (-2.54, 1.78)
- moved C13 14.0 mm to (-14.7, 2.82)
- moved C14 14.0 mm to (-14.6, 4.75)
- moved C12 13.9 mm to (-2.59, 5.97)
- moved C15 13.5 mm to (-14.7, 10.3)
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Connections:
- removed net SW0_GND: C17.1, C18.1, U3.1, U3.5, U3.7
- net SCL: now also R4.1, U4.6
- net SDA: now also R5.1, U4.3
- net SW0_VCC: now also C19.2, R4.2, R5.2, U4.1, U4.5
- net SW1_GND: now also C17.1, C18.1, C19.1, U3.1, U3.5, U3.7, U4.2, U4.4, U4.DIEPAD
Routing:
- net SW0_VCC: track 0.00 -> 70.7 mm, vias 0 -> 3
- net V_BATT: track 0.00 -> 66.5 mm
- net SW1_GND: track 0.00 -> 58.0 mm, vias 0 -> 4
- net TX: track 0.00 -> 44.3 mm
- net SDA: track 0.00 -> 35.6 mm, vias 0 -> 2
- net RX: track 0.00 -> 35.2 mm
- net EFUSE: track 0.00 -> 32.3 mm, vias 0 -> 2
- net SCL: track 0.00 -> 32.0 mm, vias 0 -> 3
- net N$3: track 0.00 -> 26.6 mm, vias 0 -> 2
- net VIN: track 0.00 -> 23.0 mm, vias 0 -> 1
- net VCC: track 0.00 -> 17.6 mm, vias 0 -> 3
- net VCC_1: track 0.00 -> 13.9 mm
- net N$7: track 0.00 -> 10.2 mm
- net XOUT: track 0.00 -> 9.66 mm
- net N$8: track 0.00 -> 8.89 mm
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Other:
- board text added: "Garden Stake"
- board text removed: "Purple Daisy IN100"
