File: magnet.sch (EAGLE design)
At the start: 37 parts, among them U1 IN100, U2 LTC3106EFE#PBF, U3 BME280, U4 SGP30, Y1 CX3225SB26000D0FLJCC, Y2 ECS-.327-12.5-16-TR

Commit message: File check-in
Parts:
- added C19: 100nF, OPL_Capacitor:CERAMIC-100NF-50V-10%-X7R(0603)
- added H1: MOUNT-HOLE3.0, holes:MOUNT-HOLE3.0
- added R4, R5: 2.2K, SparkFun-Resistors:2.2KOHM-0603-1/10W-1%
Connections:
- removed net SW0_GND: C17.1, C18.1, U3.GND, U3.SDO
- net SCL: now also R4.1, U4.SCL
- net SDA: now also R5.1, U4.SDA
- net SW0_VCC: now also C19.2, R4.2, R5.2, U4.VDD, U4.VDDH
- net SW1_GND: now also C17.1, C18.1, C19.1, U3.GND, U3.SDO, U4.DIEPAD, U4.R, U4.VSS
Other:
- moved on the sheet: U4
Changed lines of the file:
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@@
 <part name="C17" library="OPL_Capacitor" library_urn="urn:adsk.eagle:library:8004261" deviceset="CERAMIC-100NF-50V-10%-X7R(0603)" device="" package3d_urn="urn:adsk.eagle:package:8004287/1" value="100nF"/>
 <part name="C18" library="OPL_Capacitor" library_urn="urn:adsk.eagle:library:8004261" deviceset="CERAMIC-100NF-50V-10%-X7R(0603)" device="" package3d_urn="urn:adsk.eagle:package:8004287/1" value="100nF"/>
+<part name="C19" library="OPL_Capacitor" library_urn="urn:adsk.eagle:library:8004261" deviceset="CERAMIC-100NF-50V-10%-X7R(0603)" device="" package3d_urn="urn:adsk.eagle:package:8004287/1" value="100nF"/>
+<part name="H1" library="holes" library_urn="urn:adsk.eagle:library:237" deviceset="MOUNT-HOLE" device="3.0" package3d_urn="urn:adsk.eagle:package:14277/1"/>
+<part name="R4" library="SparkFun-Resistors" library_urn="urn:adsk.eagle:library:532" deviceset="2.2KOHM" device="-0603-1/10W-1%" package3d_urn="urn:adsk.eagle:package:39650/1" value="2.2K"/>
+<part name="R5" library="SparkFun-Resistors" library_urn="urn:adsk.eagle:library:532" deviceset="2.2KOHM" device="-0603-1/10W-1%" package3d_urn="urn:adsk.eagle:package:39650/1" value="2.2K"/>
 </parts>
 <sheets>
@@
 <attribute name="VALUE" x="206.4937" y="145.0216" size="1.27" layer="96" font="vector" ratio="20"/>
 </instance>
-<instance part="U4" gate="G$1" x="170.18" y="53.34" smashed="yes">
-<attribute name="NAME" x="162.56" y="61.468" size="1.778" layer="95" font="vector" ratio="20"/>
-<attribute name="VALUE" x="172.72" y="61.214" size="1.27" layer="96" font="vector" ratio="20"/>
+<instance part="U4" gate="G$1" x="215.9" y="88.9" smashed="yes">
+<attribute name="NAME" x="208.28" y="97.028" size="1.778" layer="95" font="vector" ratio="20"/>
+<attribute name="VALUE" x="218.44" y="96.774" size="1.27" layer="96" font="vector" ratio="20"/>
 </instance>
 <instance part="C17" gate="G$1" x="226.568" y="132.588" smashed="yes" rot="R90">
@@
 <attribute name="NAME" x="228.854" y="128.778" size="1.27" layer="95" font="vector" ratio="20" rot="R90"/>
 <attribute name="VALUE" x="228.854" y="133.604" size="1.27" layer="96" font="vector" ratio="20" rot="R90"/>
+</instance>
+<instance part="C19" gate="G$1" x="184.912" y="89.154" smashed="yes" rot="R90">
+<attribute name="NAME" x="184.658" y="85.344" size="1.27" layer="95" font="vector" ratio="20" rot="R90"/>
+<attribute name="VALUE" x="184.658" y="90.17" size="1.27" layer="96" font="vector" ratio="20" rot="R90"/>
+</instance>
+<instance part="H1" gate="G$1" x="246.634" y="23.368" smashed="yes">
+<attribute name="NAME" x="248.666" y="23.9522" size="1.27" layer="95" font="vector" ratio="20"/>
+<attribute name="VALUE" x="248.666" y="20.9042" size="1.016" layer="96" font="vector" display="off"/>
+</instance>
+<instance part="R4" gate="G$1" x="170.18" y="139.7" smashed="yes" rot="R90">
+<attribute name="NAME" x="169.164" y="144.272" size="1.27" layer="95" font="vector" ratio="20" rot="R180" align="bottom-center"/>
+<attribute name="VALUE" x="168.148" y="135.382" size="1.27" layer="96" font="vector" ratio="20" rot="R180" align="top-center"/>
+</instance>
+<instance part="R5" gate="G$1" x="172.72" y="139.7" smashed="yes" rot="R90">
+<attribute name="NAME" x="174.244" y="144.526" size="1.27" layer="95" font="vector" ratio="20" rot="R180" align="bottom-center"/>
+<attribute name="VALUE" x="175.006" y="135.382" size="1.27" layer="96" font="vector" ratio="20" rot="R180" align="top-center"/>
 </instance>
 </instances>
@@
 <wire x1="229.108" y1="139.7" x2="226.568" y2="139.7" width="0.1524" layer="91"/>
 <junction x="226.568" y="139.7"/>
+<pinref part="R5" gate="G$1" pin="2"/>
+<wire x1="172.72" y1="144.78" x2="172.72" y2="154.94" width="0.1524" layer="91"/>
+<wire x1="172.72" y1="154.94" x2="180.34" y2="154.94" width="0.1524" layer="91"/>
+<junction x="180.34" y="154.94"/>
+<pinref part="R4" gate="G$1" pin="2"/>
+<wire x1="170.18" y1="144.78" x2="170.18" y2="154.94" width="0.1524" layer="91"/>
+<wire x1="170.18" y1="154.94" x2="172.72" y2="154.94" width="0.1524" layer="91"/>
+<junction x="172.72" y="154.94"/>
+</segment>
+<segment>
+<pinref part="U4" gate="G$1" pin="VDD"/>
+<wire x1="205.74" y1="93.98" x2="200.66" y2="93.98" width="0.1524" layer="91"/>
+<pinref part="U4" gate="G$1" pin="VDDH"/>
+<wire x1="205.74" y1="91.44" x2="200.66" y2="91.44" width="0.1524" layer="91"/>
+<wire x1="200.66" y1="91.44" x2="200.66" y2="93.98" width="0.1524" layer="91"/>
+<junction x="200.66" y="93.98"/>
+<label x="197.104" y="95.504" size="1.27" layer="95" font="vector" ratio="20" rot="R180"/>
+<pinref part="C19" gate="G$1" pin="2"/>
+<wire x1="184.912" y1="92.964" x2="184.912" y2="93.98" width="0.1524" layer="91"/>
+<wire x1="184.912" y1="93.98" x2="200.66" y2="93.98" width="0.1524" layer="91"/>
 </segment>
 </net>
@@
 <label x="91.44" y="119.38" size="1.27" layer="95" font="vector" ratio="20" xref="yes"/>
 </segment>
-</net>
-<net name="SW0_GND" class="0">
+<segment>
+<pinref part="U4" gate="G$1" pin="DIEPAD"/>
+<wire x1="205.74" y1="83.82" x2="200.66" y2="83.82" width="0.1524" layer="91"/>
+<pinref part="U4" gate="G$1" pin="VSS"/>
+<wire x1="205.74" y1="86.36" x2="200.66" y2="86.36" width="0.1524" layer="91"/>
+<wire x1="200.66" y1="86.36" x2="200.66" y2="83.82" width="0.1524" layer="91"/>
+<junction x="200.66" y="83.82"/>
+<pinref part="U4" gate="G$1" pin="R"/>
+<wire x1="205.74" y1="88.9" x2="200.66" y2="88.9" width="0.1524" layer="91"/>
+<wire x1="200.66" y1="88.9" x2="200.66" y2="86.36" width="0.1524" layer="91"/>
+<junction x="200.66" y="86.36"/>
+<label x="197.358" y="85.09" size="1.27" layer="95" font="vector" ratio="20" rot="R180"/>
+<pinref part="C19" gate="G$1" pin="1"/>
+<wire x1="184.912" y1="85.344" x2="184.912" y2="83.82" width="0.1524" layer="91"/>
+<wire x1="184.912" y1="83.82" x2="200.66" y2="83.82" width="0.1524" layer="91"/>
+</segment>
 <segment>
 <pinref part="U3" gate="G$1" pin="GND"/>
@@
 <segment>
 <pinref part="U3" gate="G$1" pin="SCK"/>
-<wire x1="187.96" y1="132.08" x2="167.64" y2="132.08" width="0.1524" layer="91"/>
+<wire x1="187.96" y1="132.08" x2="170.18" y2="132.08" width="0.1524" layer="91"/>
 <label x="167.64" y="132.08" size="1.27" layer="95" font="vector" ratio="20" rot="R180" xref="yes"/>
+<pinref part="R4" gate="G$1" pin="1"/>
+<wire x1="170.18" y1="132.08" x2="167.64" y2="132.08" width="0.1524" layer="91"/>
+<wire x1="170.18" y1="134.62" x2="170.18" y2="132.08" width="0.1524" layer="91"/>
+<junction x="170.18" y="132.08"/>
+</segment>
+<segment>
+<pinref part="U4" gate="G$1" pin="SCL"/>
+<wire x1="226.06" y1="86.36" x2="231.14" y2="86.36" width="0.1524" layer="91"/>
+<label x="231.14" y="86.36" size="1.27" layer="95" font="vector" ratio="20" xref="yes"/>
 </segment>
 </net>
@@
 <segment>
 <pinref part="U3" gate="G$1" pin="SDI"/>
-<wire x1="187.96" y1="129.54" x2="167.64" y2="129.54" width="0.1524" layer="91"/>
+<wire x1="187.96" y1="129.54" x2="172.72" y2="129.54" width="0.1524" layer="91"/>
 <label x="167.64" y="129.54" size="1.27" layer="95" font="vector" ratio="20" rot="R180" xref="yes"/>
-</segment>
-</net>
+<pinref part="R5" gate="G$1" pin="1"/>
+<wire x1="172.72" y1="129.54" x2="167.64" y2="129.54" width="0.1524" layer="91"/>
+<wire x1="172.72" y1="134.62" x2="172.72" y2="129.54" width="0.1524" layer="91"/>
+<junction x="172.72" y="129.54"/>
+</segment>
+<segment>
+<pinref part="U4" gate="G$1" pin="SDA"/>
+<wire x1="226.06" y1="91.44" x2="231.14" y2="91.44" width="0.1524" layer="91"/>
+<label x="231.14" y="91.44" size="1.27" layer="95" font="vector" ratio="20"/>
+</segment>
+</net>
